File: Drakula.sch (EAGLE design)
At the start: 72 parts, among them IC1 STM32F405RGT6, IC2 USBLC6-2SC6, IC3 AMS1117-3.3V, IC4 ESP32-S2-WROOM-I_M22S2H3200UH3, IC5 USBLC6-2SC6, IC6 CP2102, Q1 PMOSFET, X1 1751248, Y1 FC-135R_32.7680KA-A0

Commit message: added max485
Parts:
- added C27: 10u, rcl:C-EUC0603
- added C28: 1u, rcl:C-EUC0603
- added C29, C30: 22u, rcl:C-EUC0805
- added IC7: MAX485ESA+, MAX485ESA+:MAX485ESA+
- added IC8: 5VREGULATOR, NCV2931AST-5T3G:5VREGULATOR
- added LED2: (no value), adafruit:LEDCHIPLED_0603
- added R21: 120, rcl:R-EU_R0603
- added R22, R23: 20k, rcl:R-EU_R0603
- added R24, R25, R26, R27: 10k, rcl:R-EU_R0603
- added R28: 1k, rcl:R-EU_R0603
- added X2: 1751248, con-phoenix-350:1751248
Connections:
- new net +5V: C27.1, C28.1, C29.1, IC7.VCC, IC8.OUTPUT, R23.2, R24.2, R25.2, R26.2, R27.2, R28.2
- new net N$27: IC7.!RE, R26.1
- new net N$28: IC7.RO, R27.1
- new net N$33: LED2.A, R28.1
- new net N$7: IC7.DI, R24.1
- new net N$9: IC7.DE, R25.1
- new net RS485_A: IC7.A, R21.1, R23.1, X2-1.K
- new net RS485_B: IC7.B, R21.2, R22.1, X2-2.K
- net GND: now also C27.2, C28.2, C29.2, C30.1, IC7.GND, IC8.GROUND_1, LED2.C, R22.2
- net VIN: now also C30.2, IC8.INPUT

Commit message: done schematic
Parts:
- added C31, C32: 18p, rcl:C-EUC0603
- added C33: 22u, rcl:C-EUC0805
- added C34: 100n, rcl:C-EUC0805
- added C35: 1u, rcl:C-EUC0603
- added C36, C39, C41, C42: 10n, rcl:C-EUC0603
- added C37, C40: 6.8n, rcl:C-EUC0603
- added C38: 4.7u, rcl:C-EUC0603
- added C43: 1n, rcl:C-EUC0603
- added C44, C45, C46, C47, C48, C49: 100n, rcl:C-EUC0603
- added C50: 10u, rcl:C-EUC0603
- added FB4: 742792651, ferrite bead:742792651
- added IC9: W5500, W5500:W5500
- added J1: J1B1211CCD, rj45:J1B1211CCD
- added R29: 1M, rcl:R-EU_R0603
- added R30: 12.4k, rcl:R-EU_R0603
- added R31, R32, R33, R35, R42, R43: 0R, rcl:R-EU_R0603
- added R34, R36, R37, R38, R39: 49.9R, rcl:R-EU_R0603
- added R40, R41: 330R, rcl:R-EU_R0603
- added Y2: ABM3-25.000MHZ-B2-T, ABM3-25.000MHZ-B2-T:ABM3-25.000MHZ-B2-T
Connections:
- removed net N$27: IC7.!RE, R26.1
- removed net N$28: IC7.RO, R27.1
- removed net N$7: IC7.DI, R24.1
- removed net N$9: IC7.DE, R25.1
- new net 3V3A: C35.1, C36.1, C44.2, C45.2, C46.2, C47.2, C48.2, C49.2, C50.2, FB4.2, IC9.AVDD_1, IC9.AVDD_2, IC9.AVDD_3, IC9.AVDD_4, IC9.AVDD_5, IC9.AVDD_6, R37.2, R38.2, R39.2
- new net ACTLED: IC9.ACTLED, R40.1
- new net DD: IC1.PB1, IC7.!RE, IC7.DE, R25.1, R26.1
- new net DI: IC7.DI, R24.1, R43.1
- new net INTN: IC9.INTN
- new net LINKLED: IC9.LINKLED, R41.1
- new net MISO: IC1.PC11, IC9.MISO
- new net MOSI: IC1.PB5, IC9.MOSI
- new net N$31: C39.2, IC9.1V2O
- new net N$32: C38.2, IC9.TOCAP
- new net N$34: IC9.EXRES1, R30.1
- new net N$35: IC9.TXN, R31.1
- new net N$36: IC9.TXP, R32.1
- new net N$37: IC9.RXN, R33.1
- new net N$38: IC9.RXP, R35.1
- new net N$39: J1.1, R32.2, R38.1
- new net N$40: J1.3, R31.2, R37.1
- new net N$41: C40.2, J1.6
- new net N$42: C37.2, J1.4
- new net N$43: C37.1, R34.2, R35.2
- new net N$44: C40.1, R33.2, R36.2
- new net N$45: C41.1, J1.5, R34.1, R36.1
- new net N$46: J1.9, R40.2
- new net N$47: C42.2, J1.2, R39.1
- new net N$48: J1.11, R41.2
- new net RO: IC7.RO, R27.1, R42.1
- new net RSTN: IC9.RSTN
- new net SCLK: IC1.PC10, IC9.SCLK
- new net SCSN: IC1.PB0, IC9.SCSN
- new net UART5_RX: IC1.PD2, R42.2
- new net UART5_TX: IC1.PC12, R43.2
- new net VSS: C43.2, J1.13, J1.14, J1.8
- new net XI: C31.2, IC9.XI/CLKIN, R29.2, Y2.2
- new net XO: C32.2, IC9.XO, R29.1, Y2.1
- net +3V3: now also C33.1, C34.1, FB4.1, IC9.PMODE0, IC9.PMODE1, IC9.PMODE2, IC9.VDD, J1.10, J1.12
- net GND: now also C31.1, C32.1, C33.2, C34.2, C35.2, C36.2, C38.1, C39.1, C41.2, C42.1, C43.1, C44.1, C45.1, C46.1, C47.1, C48.1, C49.1, C50.1, IC9.AGND_1, IC9.AGND_2, IC9.AGND_3, IC9.AGND_4, IC9.AGND_5, IC9.AGND_6, IC9.GND, R30.2
Other:
- moved on the sheet: C6, C7, FB1

Commit message: added doc with product description
Parts:
- removed C22, C46, C47, C48, C49: 100n, rcl:C-EUC0603
- removed C27, C50: 10u, rcl:C-EUC0603
- removed R25: 10k, rcl:R-EU_R0603
- added J2: 61300411121, Headers:61300411121
Connections:
- net +3V3: no longer C22.1
- net +5V: no longer C27.1, R25.2
- net 3V3A: no longer C46.2, C47.2, C48.2, C49.2, C50.2
- net CLK: now also J2.4
- net DD: now also IC1.PA14; no longer IC1.PB1, R25.1
- net GND: no longer C22.2, C27.2, C46.1, C47.1, C48.1, C49.1, C50.1
- net LED_B: now also IC1.PB12; no longer IC1.PB14
- net LED_G: now also IC1.PB14; no longer IC1.PB12
- net TDI: now also J2.2
- net TDO: now also J2.3
- net TMS: now also J2.1
